File: projects/hukuzawa/Motordriver/MD2017_Ctrl.sch (EAGLE design)
At the start: 5 parts, among them IC1 PIC16F648, J1 3X1A, J2 3X1A, Q1 CERALOCK

Commit message: 回路図作業途中
Parts:
- added U$1, U$2, U$3: 8PIN, FH105:8PIN
Changed lines of the file:
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@@
 <setting verticaltext="up"/>
 </settings>
-<grid distance="0.1" unitdist="inch" unit="mil" style="lines" multiple="1" display="no" altdistance="0.01" altunitdist="inch" altunit="mil"/>
+<grid distance="0.1" unitdist="inch" unit="inch" style="lines" multiple="1" display="no" altdistance="0.01" altunitdist="inch" altunit="inch"/>
 <layers>
 <layer number="1" name="Top" color="4" fill="1" visible="no" active="no"/>
@@
 <part name="Q1" library="FP-21T for MITS" deviceset="CERALOCK" device=""/>
 <part name="NJM1" library="My_NJM7805" deviceset="NJM7805" device=""/>
+<part name="U$1" library="FH105" deviceset="8PIN" device=""/>
+<part name="U$2" library="FH105" deviceset="8PIN" device=""/>
+<part name="U$3" library="FH105" deviceset="8PIN" device=""/>
 </parts>
 <sheets>
@@
 <instance part="Q1" gate="G$1" x="-2.54" y="5.08" rot="R90"/>
 <instance part="NJM1" gate="G$1" x="-66.04" y="48.26"/>
+<instance part="U$1" gate="-3" x="27.94" y="-15.24"/>
+<instance part="U$1" gate="-4" x="27.94" y="-20.32"/>
+<instance part="U$1" gate="-5" x="27.94" y="-25.4"/>
+<instance part="U$1" gate="-6" x="27.94" y="-30.48"/>
+<instance part="U$1" gate="-2" x="27.94" y="-10.16"/>
+<instance part="U$1" gate="-8" x="27.94" y="-40.64"/>
+<instance part="U$1" gate="-7" x="27.94" y="-35.56"/>
+<instance part="U$1" gate="-1" x="27.94" y="-5.08"/>
+<instance part="U$2" gate="-3" x="66.04" y="-15.24"/>
+<instance part="U$2" gate="-4" x="66.04" y="-20.32"/>
+<instance part="U$2" gate="-5" x="66.04" y="-25.4"/>
+<instance part="U$2" gate="-6" x="66.04" y="-30.48"/>
+<instance part="U$2" gate="-2" x="66.04" y="-10.16"/>
+<instance part="U$2" gate="-8" x="66.04" y="-40.64"/>
+<instance part="U$2" gate="-7" x="66.04" y="-35.56"/>
+<instance part="U$2" gate="-1" x="66.04" y="-5.08"/>
+<instance part="U$3" gate="-3" x="83.82" y="-15.24"/>
+<instance part="U$3" gate="-4" x="83.82" y="-20.32"/>
+<instance part="U$3" gate="-5" x="83.82" y="-25.4"/>
+<instance part="U$3" gate="-6" x="83.82" y="-30.48"/>
+<instance part="U$3" gate="-2" x="83.82" y="-10.16"/>
+<instance part="U$3" gate="-8" x="83.82" y="-40.64"/>
+<instance part="U$3" gate="-7" x="83.82" y="-35.56"/>
+<instance part="U$3" gate="-1" x="83.82" y="-5.08"/>
 </instances>
 <busses>
