File: projects/KatouRyuhei/Renshu/ENZANKI/ENZANKI.sch (EAGLE design)
At the start: 13 parts

Commit message: 回路図の作成
作成途中
Parts:
- added R10, R11, R5, R9: (no value), rcl:R-EU_R3216W
Connections:
- new net GND: S1.2, S2.2, S3.2, S4.2, U$1.VSS1
- new net N$1: LED1.A, R1.2
- new net N$2: LED2.A, R2.2
- new net N$3: LED3.A, R3.2
- new net N$4: LED4.A, R4.2
- new net N$5: R5.1, S1.3
- new net N$6: R9.1, S2.3
- new net N$7: R10.1, S3.3
- new net N$8: R11.1, S4.3
- new net VDD: R1.1, R10.2, R11.2, R2.1, R3.1, R4.1, R5.2, R9.2, U$1.VDD
Other:
- moved on the sheet: S1, S2, S3, S4
Changed lines of the file:
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@@
 <layer number="51" name="tDocu" color="7" fill="1" visible="no" active="no"/>
 <layer number="52" name="bDocu" color="7" fill="1" visible="no" active="no"/>
+<layer number="53" name="tGND_GNDA" color="7" fill="9" visible="no" active="no"/>
+<layer number="54" name="bGND_GNDA" color="1" fill="9" visible="no" active="no"/>
 <layer number="91" name="Nets" color="2" fill="1" visible="yes" active="yes"/>
 <layer number="92" name="Busses" color="1" fill="1" visible="yes" active="yes"/>
@@
 <part name="R3" library="rcl" deviceset="R-EU_" device="R3216W"/>
 <part name="R4" library="rcl" deviceset="R-EU_" device="R3216W"/>
+<part name="VDD1" library="supply1" deviceset="VDD" device=""/>
+<part name="VDD2" library="supply1" deviceset="VDD" device=""/>
+<part name="GND1" library="supply1" deviceset="GND" device=""/>
+<part name="R5" library="rcl" deviceset="R-EU_" device="R3216W"/>
+<part name="GND2" library="supply1" deviceset="GND" device=""/>
+<part name="R9" library="rcl" deviceset="R-EU_" device="R3216W"/>
+<part name="GND3" library="supply1" deviceset="GND" device=""/>
+<part name="R10" library="rcl" deviceset="R-EU_" device="R3216W"/>
+<part name="GND4" library="supply1" deviceset="GND" device=""/>
+<part name="R11" library="rcl" deviceset="R-EU_" device="R3216W"/>
+<part name="GND5" library="supply1" deviceset="GND" device=""/>
+<part name="VDD3" library="supply1" deviceset="VDD" device=""/>
+<part name="VDD4" library="supply1" deviceset="VDD" device=""/>
+<part name="VDD5" library="supply1" deviceset="VDD" device=""/>
+<part name="VDD6" library="supply1" deviceset="VDD" device=""/>
+<part name="VDD7" library="supply1" deviceset="VDD" device=""/>
+<part name="VDD8" library="supply1" deviceset="VDD" device=""/>
+<part name="VDD9" library="supply1" deviceset="VDD" device=""/>
 </parts>
 <sheets>
@@
 <instances>
 <instance part="U$1" gate="IC" x="-10.16" y="55.88"/>
-<instance part="S1" gate="1" x="35.56" y="30.48" rot="R270"/>
-<instance part="S2" gate="1" x="50.8" y="30.48" rot="R270"/>
-<instance part="S3" gate="1" x="66.04" y="30.48" rot="R270"/>
-<instance part="S4" gate="1" x="81.28" y="30.48" rot="R270"/>
+<instance part="S1" gate="1" x="35.56" y="10.16"/>
+<instance part="S2" gate="1" x="50.8" y="10.16"/>
+<instance part="S3" gate="1" x="66.04" y="10.16"/>
+<instance part="S4" gate="1" x="81.28" y="10.16"/>
 <instance part="LED1" gate="G$1" x="68.58" y="86.36" rot="R90"/>
 <instance part="LED2" gate="G$1" x="68.58" y="76.2" rot="R90"/>
@@
 <instance part="R3" gate="G$1" x="58.42" y="66.04"/>
 <instance part="R4" gate="G$1" x="58.42" y="55.88"/>
+<instance part="VDD1" gate="G$1" x="-40.64" y="60.96" rot="R90"/>
+<instance part="VDD2" gate="G$1" x="48.26" y="55.88" rot="R90"/>
+<instance part="GND1" gate="1" x="-40.64" y="50.8" rot="R270"/>
+<instance part="R5" gate="G$1" x="38.1" y="22.86" rot="R90"/>
+<instance part="GND2" gate="1" x="35.56" y="0"/>
+<instance part="R9" gate="G$1" x="53.34" y="22.86" rot="R90"/>
+<instance part="GND3" gate="1" x="50.8" y="0"/>
+<instance part="R10" gate="G$1" x="68.58" y="22.86" rot="R90"/>
+<instance part="GND4" gate="1" x="66.04" y="0"/>
+<instance part="R11" gate="G$1" x="83.82" y="22.86" rot="R90"/>
+<instance part="GND5" gate="1" x="81.28" y="0"/>
+<instance part="VDD3" gate="G$1" x="38.1" y="33.02"/>
+<instance part="VDD4" gate="G$1" x="53.34" y="33.02"/>
+<instance part="VDD5" gate="G$1" x="68.58" y="33.02"/>
+<instance part="VDD6" gate="G$1" x="83.82" y="33.02"/>
+<instance part="VDD7" gate="G$1" x="48.26" y="86.36" rot="R90"/>
+<instance part="VDD8" gate="G$1" x="48.26" y="76.2" rot="R90"/>
+<instance part="VDD9" gate="G$1" x="48.26" y="66.04" rot="R90"/>
 </instances>
 <busses>
 </busses>
 <nets>
+<net name="VDD" class="0">
+<segment>
+<pinref part="VDD1" gate="G$1" pin="VDD"/>
+<pinref part="U$1" gate="IC" pin="VDD"/>
+<wire x1="-38.1" y1="60.96" x2="-35.56" y2="60.96" width="0.1524" layer="91"/>
+</segment>
+<segment>
+<pinref part="VDD3" gate="G$1" pin="VDD"/>
+<pinref part="R5" gate="G$1" pin="2"/>
+<wire x1="38.1" y1="30.48" x2="38.1" y2="27.94" width="0.1524" layer="91"/>
+</segment>
+<segment>
+<pinref part="VDD4" gate="G$1" pin="VDD"/>
+<pinref part="R9" gate="G$1" pin="2"/>
+<wire x1="53.34" y1="30.48" x2="53.34" y2="27.94" width="0.1524" layer="91"/>
+</segment>
+<segment>
+<pinref part="VDD5" gate="G$1" pin="VDD"/>
+<pinref part="R10" gate="G$1" pin="2"/>
+<wire x1="68.58" y1="30.48" x2="68.58" y2="27.94" width="0.1524" layer="91"/>
+</segment>
+<segment>
+<pinref part="VDD6" gate="G$1" pin="VDD"/>
+<pinref part="R11" gate="G$1" pin="2"/>
+<wire x1="83.82" y1="30.48" x2="83.82" y2="27.94" width="0.1524" layer="91"/>
+</segment>
+<segment>
+<pinref part="VDD9" gate="G$1" pin="VDD"/>
+<pinref part="R3" gate="G$1" pin="1"/>
+<wire x1="50.8" y1="66.04" x2="53.34" y2="66.04" width="0.1524" layer="91"/>
+</segment>
+<segment>
+<pinref part="VDD2" gate="G$1" pin="VDD"/>
+<pinref part="R4" gate="G$1" pin="1"/>
+<wire x1="50.8" y1="55.88" x2="53.34" y2="55.88" width="0.1524" layer="91"/>
+</segment>
+<segment>
+<pinref part="VDD8" gate="G$1" pin="VDD"/>
+<pinref part="R2" gate="G$1" pin="1"/>
+<wire x1="50.8" y1="76.2" x2="53.34" y2="76.2" width="0.1524" layer="91"/>
+</segment>
+<segment>
+<pinref part="VDD7" gate="G$1" pin="VDD"/>
+<pinref part="R1" gate="G$1" pin="1"/>
+<wire x1="50.8" y1="86.36" x2="53.34" y2="86.36" width="0.1524" layer="91"/>
+</segment>
+</net>
+<net name="GND" class="0">
+<segment>
+<pinref part="GND1" gate="1" pin="GND"/>
+<pinref part="U$1" gate="IC" pin="VSS1"/>
+<wire x1="-38.1" y1="50.8" x2="-35.56" y2="50.8" width="0.1524" layer="91"/>
+</segment>
+<segment>
+<pinref part="S4" gate="1" pin="2"/>
+<pinref part="GND5" gate="1" pin="GND"/>
+<wire x1="81.28" y1="5.08" x2="81.28" y2="2.54" width="0.1524" layer="91"/>
+</segment>
+<segment>
+<pinref part="S3" gate="1" pin="2"/>
+<pinref part="GND4" gate="1" pin="GND"/>
+<wire x1="66.04" y1="5.08" x2="66.04" y2="2.54" width="0.1524" layer="91"/>
+</segment>
+<segment>
+<pinref part="S2" gate="1" pin="2"/>
+<pinref part="GND3" gate="1" pin="GND"/>
+<wire x1="50.8" y1="5.08" x2="50.8" y2="2.54" width="0.1524" layer="91"/>
+</segment>
+<segment>
+<pinref part="S1" gate="1" pin="2"/>
+<pinref part="GND2" gate="1" pin="GND"/>
+<wire x1="35.56" y1="5.08" x2="35.56" y2="2.54" width="0.1524" layer="91"/>
+</segment>
+</net>
+<net name="N$1" class="0">
+<segment>
+<pinref part="R1" gate="G$1" pin="2"/>
+<pinref part="LED1" gate="G$1" pin="A"/>
+<wire x1="63.5" y1="86.36" x2="66.04" y2="86.36" width="0.1524" layer="91"/>
+</segment>
+</net>
+<net name="N$2" class="0">
+<segment>
+<pinref part="R2" gate="G$1" pin="2"/>
+<pinref part="LED2" gate="G$1" pin="A"/>
+<wire x1="63.5" y1="76.2" x2="66.04" y2="76.2" width="0.1524" layer="91"/>
+</segment>
+</net>
+<net name="N$3" class="0">
+<segment>
+<pinref part="R3" gate="G$1" pin="2"/>
+<pinref part="LED3" gate="G$1" pin="A"/>
+<wire x1="63.5" y1="66.04" x2="66.04" y2="66.04" width="0.1524" layer="91"/>
+</segment>
+</net>
+<net name="N$4" class="0">
+<segment>
+<pinref part="R4" gate="G$1" pin="2"/>
+<pinref part="LED4" gate="G$1" pin="A"/>
+<wire x1="63.5" y1="55.88" x2="66.04" y2="55.88" width="0.1524" layer="91"/>
+</segment>
+</net>
+<net name="N$5" class="0">
+<segment>
+<pinref part="R5" gate="G$1" pin="1"/>
+<pinref part="S1" gate="1" pin="3"/>
+<wire x1="38.1" y1="17.78" x2="38.1" y2="15.24" width="0.1524" layer="91"/>
+</segment>
+</net>
+<net name="N$6" class="0">
+<segment>
+<pinref part="R9" gate="G$1" pin="1"/>
+<pinref part="S2" gate="1" pin="3"/>
+<wire x1="53.34" y1="17.78" x2="53.34" y2="15.24" width="0.1524" layer="91"/>
+</segment>
+</net>
+<net name="N$7" class="0">
+<segment>
+<pinref part="R10" gate="G$1" pin="1"/>
+<pinref part="S3" gate="1" pin="3"/>
+<wire x1="68.58" y1="17.78" x2="68.58" y2="15.24" width="0.1524" layer="91"/>
+</segment>
+</net>
+<net name="N$8" class="0">
+<segment>
+<pinref part="R11" gate="G$1" pin="1"/>
+<pinref part="S4" gate="1" pin="3"/>
+<wire x1="83.82" y1="17.78" x2="83.82" y2="15.24" width="0.1524" layer="91"/>
+</segment>
+</net>
 </nets>
 </sheet>

Commit message: 演算機の回路図の作成
製作途中
Parts:
- removed R11: (no value), rcl:R-EU_R3216W
- added H1, H2, H3, H4: HOLE3.3M3BOLT, Hole:HOLE3.3M3BOLT
- added LED5: (no value), FP-21T for MITS:LED5MM
- added R6, R7, R8: (no value), rcl:R-EU_R3216W
- added S5: (no value), switch:SLIDESW
Connections:
- new net CHECK: LED5.C, S5.1
- new net IN1: S1.1, U$1.RA0/AN0/ULPWU/C12IN0-
- new net IN2: S2.1, U$1.RA1/AN1/C12IN1-
- new net IN3: S3.1, U$1.RA2/AN2/VREF-/CVREF/C2IN+
- new net IN4: S4.1, U$1.RA3/AN3/VREF+/C1IN+
- new net N$9: LED5.A, R10.2
- new net OUT1: LED1.C, U$1.RA4/TOCKI/C1OUT
- new net OUT2: LED2.C, U$1.RA5/AN4/!SS!/C2OUT
- new net OUT3: LED3.C, U$1.RA6/OSC2/CLKOUT
- new net OUT4: LED4.C, U$1.RA7/OSC1/CLKIN
- new net R1: R1.1, S1.3
- net GND: now also S5.2
- net N$1: now also R6.2; no longer R1.2
- net N$2: now also R7.2; no longer R2.2
- net N$3: now also R8.2; no longer R3.2
- net N$4: now also R9.2; no longer R4.2
- net N$5: now also S5.3; no longer S1.3
- net N$6: now also R2.1; no longer R9.1
- net N$7: now also R3.1; no longer R10.1
- net N$8: now also R4.1; no longer R11.1
- net VDD: now also R1.2, R10.1, R2.2, R3.2, R4.2, R6.1, R7.1, R8.1, R9.1; no longer R1.1, R10.2, R11.2, R2.1, R3.1, R4.1, R9.2
Other:
- moved on the sheet: R1, R10, R2, R3, R4, R5, R9, S1, S2, S3, S4

Commit message: 回路図の作成
Parts:
- removed R6: (no value), rcl:R-EU_R3216W
- added R11, RC: (no value), rcl:R-EU_R3216W
- added S6: (no value), switch:SLIDESW
Connections:
- new net IN5: S6.1, U$1.RA4/TOCKI/C1OUT
- new net N$10: R5.1, S6.3
- net GND: now also S6.2
- net N$1: now also R7.2; no longer R6.2
- net N$2: now also R8.2; no longer R7.2
- net N$3: now also R9.2; no longer R8.2
- net N$4: now also R10.2; no longer R9.2
- net N$5: now also RC.1; no longer R5.1
- net N$9: now also R11.2; no longer R10.2
- net OUT1: now also U$1.RA5/AN4/!SS!/C2OUT; no longer U$1.RA4/TOCKI/C1OUT
- net OUT2: now also U$1.RA6/OSC2/CLKOUT; no longer U$1.RA5/AN4/!SS!/C2OUT
- net OUT3: now also U$1.RA7/OSC1/CLKIN; no longer U$1.RA6/OSC2/CLKOUT
- net OUT4: now also U$1.RB0/AN12/INT; no longer U$1.RA7/OSC1/CLKIN
- net VDD: now also R11.1, RC.2; no longer R6.1
Other:
- moved on the sheet: H1, H2, H3, H4, LED1, LED2, LED3, LED4, LED5, R1, R10, R2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

Commit message: 回路図とボード図の作成
作成途中
Parts:
- renumbered RC to R6
Connections:
- net CHECK: now also S6.1; no longer S5.1
- net IN5: now also S5.1; no longer S6.1
- net N$10: now also S5.3; no longer S6.3
- net N$5: now also S6.3; no longer S5.3
Other:
- moved on the sheet: S5, S6
Changed lines of the file:
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@@
 <part name="R11" library="rcl" deviceset="R-EU_" device="R3216W"/>
 <part name="LED5" library="FP-21T for MITS" deviceset="LED" device="5MM"/>
-<part name="S5" library="switch" deviceset="SLIDESW" device=""/>
-<part name="RC" library="rcl" deviceset="R-EU_" device="R3216W"/>
+<part name="S6" library="switch" deviceset="SLIDESW" device=""/>
+<part name="R6" library="rcl" deviceset="R-EU_" device="R3216W"/>
 <part name="VDD11" library="supply1" deviceset="VDD" device=""/>
 <part name="GND6" library="supply1" deviceset="GND" device=""/>
 <part name="GND7" library="supply1" deviceset="GND" device=""/>
-<part name="S6" library="switch" deviceset="SLIDESW" device=""/>
+<part name="S5" library="switch" deviceset="SLIDESW" device=""/>
 <part name="R5" library="rcl" deviceset="R-EU_" device="R3216W"/>
 <part name="VDD12" library="supply1" deviceset="VDD" device=""/>
@@
 <instance part="R11" gate="G$1" x="22.86" y="2.54"/>
 <instance part="LED5" gate="G$1" x="33.02" y="2.54" rot="R90"/>
-<instance part="S5" gate="1" x="66.04" y="-30.48"/>
-<instance part="RC" gate="G$1" x="68.58" y="-17.78" rot="R90"/>
+<instance part="S6" gate="1" x="66.04" y="-30.48"/>
+<instance part="R6" gate="G$1" x="68.58" y="-17.78" rot="R90"/>
 <instance part="VDD11" gate="G$1" x="68.58" y="-7.62"/>
 <instance part="GND6" gate="1" x="66.04" y="-40.64"/>
 <instance part="GND7" gate="1" x="50.8" y="-40.64"/>
-<instance part="S6" gate="1" x="50.8" y="-30.48"/>
+<instance part="S5" gate="1" x="50.8" y="-30.48"/>
 <instance part="R5" gate="G$1" x="53.34" y="-17.78" rot="R90"/>
 <instance part="VDD12" gate="G$1" x="53.34" y="-7.62"/>
@@
 <segment>
 <pinref part="VDD11" gate="G$1" pin="VDD"/>
-<pinref part="RC" gate="G$1" pin="2"/>
+<pinref part="R6" gate="G$1" pin="2"/>
 <wire x1="68.58" y1="-10.16" x2="68.58" y2="-12.7" width="0.1524" layer="91"/>
 </segment>
@@
 </segment>
 <segment>
-<pinref part="S5" gate="1" pin="2"/>
+<pinref part="S6" gate="1" pin="2"/>
 <pinref part="GND6" gate="1" pin="GND"/>
 <wire x1="66.04" y1="-35.56" x2="66.04" y2="-38.1" width="0.1524" layer="91"/>
 </segment>
 <segment>
-<pinref part="S6" gate="1" pin="2"/>
+<pinref part="S5" gate="1" pin="2"/>
 <pinref part="GND7" gate="1" pin="GND"/>
 <wire x1="50.8" y1="-35.56" x2="50.8" y2="-38.1" width="0.1524" layer="91"/>
@@
 </segment>
 <segment>
-<pinref part="S5" gate="1" pin="1"/>
+<pinref part="S6" gate="1" pin="1"/>
 <wire x1="63.5" y1="-25.4" x2="63.5" y2="-22.86" width="0.1524" layer="91"/>
 <label x="63.5" y="-22.86" size="1.778" layer="95" rot="R90" xref="yes"/>
@@
 <net name="N$5" class="0">
 <segment>
-<pinref part="RC" gate="G$1" pin="1"/>
+<pinref part="R6" gate="G$1" pin="1"/>
+<pinref part="S6" gate="1" pin="3"/>
+<wire x1="68.58" y1="-22.86" x2="68.58" y2="-25.4" width="0.1524" layer="91"/>
+</segment>
+</net>
+<net name="N$10" class="0">
+<segment>
+<pinref part="R5" gate="G$1" pin="1"/>
 <pinref part="S5" gate="1" pin="3"/>
-<wire x1="68.58" y1="-22.86" x2="68.58" y2="-25.4" width="0.1524" layer="91"/>
-</segment>
-</net>
-<net name="N$10" class="0">
-<segment>
-<pinref part="R5" gate="G$1" pin="1"/>
-<pinref part="S6" gate="1" pin="3"/>
 <wire x1="53.34" y1="-22.86" x2="53.34" y2="-25.4" width="0.1524" layer="91"/>
 </segment>
@@
 <net name="IN5" class="0">
 <segment>
-<pinref part="S6" gate="1" pin="1"/>
+<pinref part="S5" gate="1" pin="1"/>
 <wire x1="48.26" y1="-25.4" x2="48.26" y2="-20.32" width="0.1524" layer="91"/>
 <label x="48.26" y="-20.32" size="1.778" layer="95" rot="R90" xref="yes"/>
